File: V1.5/easyhive.sch (KiCad schematic (older format))
At the start: 107 parts, among them IC1 ATSAMD21G, IC2 BQ2407X, IC3 ADS1232, IC4 DS18B20U, IC5 XC6220B331, IC7 TPS22919, J1 U.FL, K1 693043020611, P1 PKMCS, Q1 32768 Hz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

Commit message: Begin Routing
Parts:
- removed TP1, TP19: TPTP08R, easyhive:TP08R, symbol easyhive:TPTP08R
- JP10: renamed from JP?; value I2C -> USB_BC66
- JP4: value M02-JST-2MM-SMT -> AUX; footprint easyhive:1X02_2MM_Pad_only -> easyhive:1X02_2MM_klein; symbol easyhive:M02-JST-2MM-SMT -> easyhive:M02PTH-2MM
- JP9: renamed from JP?; value M02-JST-2MM-SMT -> DBG; footprint easyhive:1X02_2MM_Pad_only -> easyhive:1X02_2MM_klein; symbol easyhive:M02-JST-2MM-SMT -> easyhive:M02PTH-2MM
- U2: renamed from U?; footprint RF_GSM:Quectel_BC66 -> easyhive:Quectel_BC66
- gave numbers to parts that had none: 5
Other:
- note added: "BC66 Module"
- note removed: "SARA N3 Module"
- moved on the sheet: R6, R7, R8, R9
Changed lines of the file:
@@
 EESchema Schematic File Version 4
-LIBS:easyhive-cache
-EELAYER 26 0
+EELAYER 30 0
 EELAYER END
 $Descr User 17018 11968
@@
 Text Label 4000 3400 0    70   ~ 0
 VUSB
-Text Label 12650 9700 0    70   ~ 0
-+1V8
 Text Label 12900 2750 0    70   ~ 0
 BC66_RXD_3V3
@@
 $EndComp
 $Comp
-L easyhive:TPTP08R TP1
-U 1 1 4FABACB0
-P 13150 9700
-F 0 "TP1" V 13100 9650 59  0000 L BNN
-F 1 "TPTP08R" H 13150 9700 50  0001 C CNN
-F 2 "easyhive:TP08R" H 13150 9700 50  0001 C CNN
-F 3 "" H 13150 9700 50  0001 C CNN
-F 4 "in Stueckliste loeschen" H 13150 9700 50  0001 C CNN "Description"
-	1    13150 9700
-	0    1    1    0
-$EndComp
-$Comp
 L easyhive:TPTP08R TP6
 U 1 1 3B17FAA9
@@
 Microcontroller SAM
 Text Notes 4850 6500 0    170  ~ 0
-SARA N3 Module
+BC66 Module
 Text Notes 1100 5100 0    170  ~ 0
 Load Cell Amplifier
@@
 BC66_PWRON
 Connection ~ 10800 7800
-Wire Wire Line
-	12400 9700 13050 9700
 $Comp
 L easyhive:GND #GND0102
 U 1 1 6029D37C
-P 8800 8400
-F 0 "#GND0102" H 8800 8400 50  0001 C CNN
-F 1 "GND" H 8700 8300 59  0000 L BNN
-F 2 "" H 8800 8400 50  0001 C CNN
-F 3 "" H 8800 8400 50  0001 C CNN
-	1    8800 8400
+P 8400 8400
+F 0 "#GND0102" H 8400 8400 50  0001 C CNN
+F 1 "GND" H 8300 8300 59  0000 L BNN
+F 2 "" H 8400 8400 50  0001 C CNN
+F 3 "" H 8400 8400 50  0001 C CNN
+	1    8400 8400
 	0    -1   -1   0
 $EndComp
 Wire Wire Line
-	8250 8100 8450 8100
-Wire Wire Line
 	8800 10450 8950 10450
 Text Label 8750 10450 0    50   ~ 0
@@
 	9050 10450 8950 10450
 Connection ~ 8950 10450
-$Comp
-L easyhive:TPTP08R TP19
-U 1 1 5FCD1F38
-P 12500 9550
-F 0 "TP19" V 12450 9500 59  0000 L BNN
-F 1 "TPTP08R" H 12500 9550 50  0001 C CNN
-F 2 "easyhive:TP08R" H 12500 9550 50  0001 C CNN
-F 3 "" H 12500 9550 50  0001 C CNN
-F 4 "in Stueckliste loeschen" H 12500 9550 50  0001 C CNN "Description"
-	1    12500 9550
-	0    1    1    0
-$EndComp
 Wire Wire Line
 	2100 7600 2100 7400
@@
 	5750 7350 5750 8700
 $Comp
-L easyhive:M02-JST-2MM-SMT JP4
+L easyhive:M02PTH-2MM JP4
 U 1 1 6030887E
 P 6600 8200
 F 0 "JP4" H 6600 8350 59  0000 C CNN
-F 1 "M02-JST-2MM-SMT" H 6550 8200 59  0000 C CNN
-F 2 "easyhive:1X02_2MM_Pad_only" H 6600 8200 50  0001 C CNN
+F 1 "AUX" H 6550 8200 59  0000 C CNN
+F 2 "easyhive:1X02_2MM_klein" H 6600 8200 50  0001 C CNN
 F 3 "" H 6600 8200 50  0001 C CNN
 F 4 "in Stueckliste loeschen" H 6600 8200 50  0001 C CNN "Description"
@@
 	6900 8200 7050 8200
 $Comp
-L quectel:BC66 U?
+L quectel:BC66 U2
 U 1 1 601D979A
 P 7650 8500
-F 0 "U?" H 7950 7450 50  0000 C CNN
+F 0 "U2" H 7950 7450 50  0000 C CNN
 F 1 "BC66" H 8000 7350 50  0000 C CNN
-F 2 "RF_GSM:Quectel_BC66" H 8200 7450 50  0001 C CNN
+F 2 "easyhive:Quectel_BC66" H 8200 7450 50  0001 C CNN
 F 3 "https://www.quectel.com/UploadImage/Downlad/Quectel_BC66_Hardware_Design_V1.1.pdf" H 9350 7500 50  0001 C CNN
 	1    7650 8500
@@
 	9050 8400 9050 8200
 $Comp
-L easyhive:RESISTOR-0402 R?
+L easyhive:RESISTOR-0402 R8
 U 1 1 6039EAB1
-P 8650 8200
-F 0 "R?" H 8350 8200 59  0000 L BNN
-F 1 "22R" H 8550 8200 59  0000 L BNN
-F 2 "easyhive:C0402" H 8650 8200 50  0001 C CNN
-F 3 "" H 8650 8200 50  0001 C CNN
-	1    8650 8200
+P 8800 8200
+F 0 "R8" H 8500 8200 59  0000 L BNN
+F 1 "22R" H 8700 8200 59  0000 L BNN
+F 2 "easyhive:C0402" H 8800 8200 50  0001 C CNN
+F 3 "" H 8800 8200 50  0001 C CNN
+	1    8800 8200
 	1    0    0    -1
 $EndComp
 $Comp
-L easyhive:RESISTOR-0402 R?
+L easyhive:RESISTOR-0402 R9
 U 1 1 6039F682
-P 8650 8300
-F 0 "R?" H 8350 8300 59  0000 L BNN
-F 1 "22R" H 8550 8300 59  0000 L BNN
-F 2 "easyhive:C0402" H 8650 8300 50  0001 C CNN
-F 3 "" H 8650 8300 50  0001 C CNN
-	1    8650 8300
+P 8800 8300
+F 0 "R9" H 8500 8300 59  0000 L BNN
+F 1 "22R" H 8700 8300 59  0000 L BNN
+F 2 "easyhive:C0402" H 8800 8300 50  0001 C CNN
+F 3 "" H 8800 8300 50  0001 C CNN
+	1    8800 8300
 	1    0    0    -1
 $EndComp
 $Comp
-L easyhive:RESISTOR-0402 R?
+L easyhive:RESISTOR-0402 R7
 U 1 1 6039F914
-P 8650 8100
-F 0 "R?" H 8350 8100 59  0000 L BNN
-F 1 "22R" H 8550 8100 59  0000 L BNN
-F 2 "easyhive:C0402" H 8650 8100 50  0001 C CNN
-F 3 "" H 8650 8100 50  0001 C CNN
-	1    8650 8100
+P 8800 8100
+F 0 "R7" H 8500 8100 59  0000 L BNN
+F 1 "22R" H 8700 8100 59  0000 L BNN
+F 2 "easyhive:C0402" H 8800 8100 50  0001 C CNN
+F 3 "" H 8800 8100 50  0001 C CNN
+	1    8800 8100
 	1    0    0    -1
 $EndComp
 Wire Wire Line
-	8850 8100 9700 8100
+	9050 8200 9000 8200
 Wire Wire Line
-	9050 8200 8850 8200
+	8600 8200 8550 8200
 Wire Wire Line
-	8450 8200 8250 8200
+	9150 8300 9000 8300
 Wire Wire Line
-	9150 8300 8850 8300
-Wire Wire Line
-	8450 8300 8250 8300
-$Comp
-L easyhive:RESISTOR-0402 R?
-U 1 1 6045970B
-P 9050 7850
-F 0 "R?" H 8850 7900 59  0000 L BNN
-F 1 "10K" H 8950 7850 59  0000 L BNN
-F 2 "easyhive:C0402" H 9050 7850 50  0001 C CNN
-F 3 "" H 9050 7850 50  0001 C CNN
-	1    9050 7850
-	0    1    1    0
-$EndComp
-Wire Wire Line
-	9050 8200 9050 8050
-Connection ~ 9050 8200
-Wire Wire Line
-	9050 7650 8950 7650
-Wire Wire Line
-	8950 7650 8950 8000
-Wire Wire Line
-	8950 8000 9400 8000
-Wire Wire Line
-	8950 8000 8250 8000
-Connection ~ 8950 8000
-Wire Wire Line
-	8250 8400 8700 8400
+	8250 8400 8300 8400
 $Comp
 L easyhive:CAPACITOR-0402 C22
@@
 Connection ~ 7650 6700
 $Comp
-L easyhive:GND #GND?
+L easyhive:GND #GND065
 U 1 1 609EBE23
 P 7900 7200
-F 0 "#GND?" H 7900 7200 50  0001 C CNN
+F 0 "#GND065" H 7900 7200 50  0001 C CNN
 F 1 "GND" H 7800 7100 59  0000 L BNN
 F 2 "" H 7900 7200 50  0001 C CNN
@@
 	5600 8800 5600 8300
 $Comp
-L easyhive:DTC123JET1G Q?
+L easyhive:DTC123JET1G Q4
 U 1 1 60ADE227
 P 5300 8600
-F 0 "Q?" V 5889 8600 50  0000 C CNN
+F 0 "Q4" V 5889 8600 50  0000 C CNN
 F 1 "DTC123JET1G" V 5980 8600 50  0000 C CNN
 F 2 "easyhive:SC75_SOT416" H 5300 9200 50  0001 L CNN
@@
 	7050 9100 5600 9100
 $Comp
-L easyhive:GND #GND?
+L easyhive:GND #GND033
 U 1 1 60B0E79D
 P 4900 9100
-F 0 "#GND?" H 4900 9100 50  0001 C CNN
+F 0 "#GND033" H 4900 9100 50  0001 C CNN
 F 1 "GND" H 4800 9000 59  0000 L BNN
 F 2 "" H 4900 9100 50  0001 C CNN
@@
 	0    1    1    0
 $EndComp
-Text Label 5050 8600 0    50   ~ 0
+Text Label 5300 8600 2    50   ~ 0
 BC66_PSM
 $Comp
-L easyhive:M02-JST-2MM-SMT JP?
+L easyhive:M02PTH-2MM JP9
 U 1 1 60BFE27F
 P 6600 8500
-F 0 "JP?" H 6600 8650 59  0000 C CNN
-F 1 "M02-JST-2MM-SMT" H 6550 8500 59  0000 C CNN
-F 2 "easyhive:1X02_2MM_Pad_only" H 6600 8500 50  0001 C CNN
+F 0 "JP9" H 6600 8650 59  0000 C CNN
+F 1 "DBG" H 6550 8500 59  0000 C CNN
+F 2 "easyhive:1X02_2MM_klein" H 6600 8500 50  0001 C CNN
 F 3 "" H 6600 8500 50  0001 C CNN
 F 4 "in Stueckliste loeschen" H 6600 8500 50  0001 C CNN "Description"
@@
 Wire Wire Line
 	7750 7350 8100 7350
-Text Label 7900 7450 0    50   ~ 0
+Text Label 7950 7350 0    50   ~ 0
 +1V8
 Wire Wire Line
@@
 BC66_TXD_1V8
 $Comp
-L easyhive:GND #GND?
+L easyhive:GND #GND064
 U 1 1 60EB106D
 P 5500 11050
-F 0 "#GND?" H 5500 11050 50  0001 C CNN
+F 0 "#GND064" H 5500 11050 50  0001 C CNN
 F 1 "GND" H 5400 10950 59  0000 L BNN
 F 2 "" H 5500 11050 50  0001 C CNN
@@
 $EndComp
 $Comp
-L easyhive:+3V3 #+3V?
+L easyhive:+3V3 #+3V03
 U 1 1 60EB114C
 P 5500 11150
-F 0 "#+3V?" H 5500 11150 50  0001 C CNN
+F 0 "#+3V03" H 5500 11150 50  0001 C CNN
 F 1 "+3V3" V 5400 10950 59  0000 L BNN
 F 2 "" H 5500 11150 50  0001 C CNN
@@
 BC66_PSM
 $Comp
-L easyhive:M04PTH-2MM JP?
+L easyhive:M04PTH-2MM JP10
 U 1 1 6106C146
 P 8800 9200
-F 0 "JP?" H 8600 9530 59  0000 L BNN
-F 1 "I2C" H 8600 8900 59  0000 L BNN
+F 0 "JP10" H 8600 9530 59  0000 L BNN
+F 1 "USB_BC66" H 8600 8900 59  0000 L BNN
 F 2 "easyhive:1X04-2MM_klein" H 8800 9200 50  0001 C CNN
 F 3 "" H 8800 9200 50  0001 C CNN
@@
 Wire Wire Line
 	8600 9400 8250 9400
+$Comp
+L easyhive:RESISTOR-0402 R6
+U 1 1 6045970B
+P 8550 7850
+F 0 "R6" H 8350 7900 59  0000 L BNN
+F 1 "10K" H 8450 7850 59  0000 L BNN
+F 2 "easyhive:C0402" H 8550 7850 50  0001 C CNN
+F 3 "" H 8550 7850 50  0001 C CNN
+	1    8550 7850
+	0    1    1    0
+$EndComp
+Wire Wire Line
+	9000 8100 9700 8100
+Wire Wire Line
+	8550 7650 8700 7650
+Wire Wire Line
+	8700 7650 8700 8000
+Connection ~ 8700 8000
+Wire Wire Line
+	8700 8000 8250 8000
+Wire Wire Line
+	8550 8050 8550 8200
+Connection ~ 8550 8200
+Wire Wire Line
+	8250 8100 8600 8100
+Wire Wire Line
+	8250 8200 8550 8200
+Wire Wire Line
+	8250 8300 8600 8300
+Wire Wire Line
+	8700 8000 9400 8000
 $EndSCHEMATC

Commit message: Need verification.
-Routing done
-Silk done
-USB Mode 2 drill Pads + R10k
-open review
Parts:
- added JP11: USB_MODE, easyhive:1X02_2MM_klein, symbol easyhive:M02PTH-2MM
- added R10: 10K, easyhive:C0402, symbol easyhive:RESISTOR-0402
- JP10: footprint easyhive:1X04-2MM_klein -> easyhive:1X03-2MM_klein; symbol easyhive:M04PTH-2MM -> easyhive:M03JST-PTH
- JP4: value AUX -> UART_AUX
- JP9: value DBG -> UART_DBG
Connections:
- wire segments 416 -> 417
Changed lines of the file:
@@
 P 6600 8200
 F 0 "JP4" H 6600 8350 59  0000 C CNN
-F 1 "AUX" H 6550 8200 59  0000 C CNN
+F 1 "UART_AUX" H 6250 8350 59  0000 C CNN
 F 2 "easyhive:1X02_2MM_klein" H 6600 8200 50  0001 C CNN
 F 3 "" H 6600 8200 50  0001 C CNN
@@
 P 6600 8500
 F 0 "JP9" H 6600 8650 59  0000 C CNN
-F 1 "DBG" H 6550 8500 59  0000 C CNN
+F 1 "UART_DBG" H 6250 8650 59  0000 C CNN
 F 2 "easyhive:1X02_2MM_klein" H 6600 8500 50  0001 C CNN
 F 3 "" H 6600 8500 50  0001 C CNN
@@
 BC66_PSM
 $Comp
-L easyhive:M04PTH-2MM JP10
-U 1 1 6106C146
-P 8800 9200
-F 0 "JP10" H 8600 9530 59  0000 L BNN
-F 1 "USB_BC66" H 8600 8900 59  0000 L BNN
-F 2 "easyhive:1X04-2MM_klein" H 8800 9200 50  0001 C CNN
-F 3 "" H 8800 9200 50  0001 C CNN
-F 4 "in Stueckliste loeschen" H 8800 9200 50  0001 C CNN "Description"
-	1    8800 9200
-	-1   0    0    1
-$EndComp
-Wire Wire Line
-	8600 9100 8250 9100
-Wire Wire Line
-	8600 9200 8250 9200
-Wire Wire Line
-	8600 9300 8250 9300
-Wire Wire Line
-	8600 9400 8250 9400
-$Comp
 L easyhive:RESISTOR-0402 R6
 U 1 1 6045970B
@@
 Wire Wire Line
 	8700 8000 9400 8000
+$Comp
+L easyhive:RESISTOR-0402 R10
+U 1 1 6012B584
+P 8450 9400
+F 0 "R10" H 8250 9450 59  0000 L BNN
+F 1 "10K" H 8350 9400 59  0000 L BNN
+F 2 "easyhive:C0402" H 8450 9400 50  0001 C CNN
+F 3 "" H 8450 9400 50  0001 C CNN
+	1    8450 9400
+	1    0    0    -1
+$EndComp
+$Comp
+L easyhive:GND #GND066
+U 1 1 6012DFCC
+P 8700 9650
+F 0 "#GND066" H 8700 9650 50  0001 C CNN
+F 1 "GND" H 8600 9550 59  0000 L BNN
+F 2 "" H 8700 9650 50  0001 C CNN
+F 3 "" H 8700 9650 50  0001 C CNN
+	1    8700 9650
+	0    1    1    0
+$EndComp
+$Comp
+L easyhive:M03JST-PTH JP10
+U 1 1 6106C146
+P 9100 9200
+F 0 "JP10" H 8750 9000 59  0000 L BNN
+F 1 "USB_BC66" H 8900 8900 59  0000 L BNN
+F 2 "easyhive:1X03-2MM_klein" H 9100 9200 50  0001 C CNN
+F 3 "" H 9100 9200 50  0001 C CNN
+F 4 "in Stueckliste loeschen" H 9100 9200 50  0001 C CNN "Description"
+	1    9100 9200
+	-1   0    0    1
+$EndComp
+Wire Wire Line
+	8250 9100 8800 9100
+Wire Wire Line
+	8250 9200 8800 9200
+Wire Wire Line
+	8250 9300 8800 9300
+$Comp
+L easyhive:M02PTH-2MM JP11
+U 1 1 60390E56
+P 9100 9550
+F 0 "JP11" H 9100 9700 59  0000 C CNN
+F 1 "USB_MODE" H 8750 9500 59  0000 C CNN
+F 2 "easyhive:1X02_2MM_klein" H 9100 9550 50  0001 C CNN
+F 3 "" H 9100 9550 50  0001 C CNN
+F 4 "in Stueckliste loeschen" H 9100 9550 50  0001 C CNN "Description"
+	1    9100 9550
+	-1   0    0    1
+$EndComp
+Wire Wire Line
+	8650 9400 8800 9400
+Wire Wire Line
+	8800 9400 8800 9550
 $EndSCHEMATC

Commit message: Add schmematic.pdf
-add easyhive-schematic.pdf
-rename C22 from 100nF to 100n
-remove text from JST PH Footprint
Parts:
- C22: value 100nF -> 100n
- U2: Manufacturer (none) -> Quectel
Changed lines of the file:
@@
 Wire Notes Line
 	13000 5700 13000 9850
-Text Notes 5150 10050 0    98   ~ 0
+Text Notes 4800 10000 0    98   ~ 0
 Level Shifter 3.3V - 1.8V
 Wire Notes Line
@@
 F 2 "easyhive:Quectel_BC66" H 8200 7450 50  0001 C CNN
 F 3 "https://www.quectel.com/UploadImage/Downlad/Quectel_BC66_Hardware_Design_V1.1.pdf" H 9350 7500 50  0001 C CNN
+F 4 "Quectel" H 7650 8500 50  0001 C CNN "Manufacturer"
 	1    7650 8500
 	1    0    0    -1
@@
 P 10650 7900
 F 0 "C22" H 10710 7815 59  0000 L BNN
-F 1 "100nF" H 10710 7915 59  0000 L BNN
+F 1 "100n" H 10710 7915 59  0000 L BNN
 F 2 "easyhive:C0402" H 10650 7900 50  0001 C CNN
 F 3 "" H 10650 7900 50  0001 C CNN
